File: Capstone/Capstone.kicad_pcb (KiCad board)
At the start: 2 copper layers, 35 parts, among them SW1 SW_Push, SW2 SW_Push, SW3 SW_Push, U2 DS3231M, U3 PCF8574AP, U4 WEMOS_D1_mini

Commit message: First Commit
Parts:
- removed BUTTON1: Button, Connector_PinHeader_2.54mm:PinHeader_1x04_P2.54mm_Vertical
- removed I2C1: I2C, Connector_PinHeader_2.54mm:PinHeader_1x04_P2.54mm_Vertical
- removed LM2596_E1: LM2596, Connector_PinHeader_2.54mm:PinHeader_1x04_P2.54mm_Vertical
- removed SERIAL1: Serial, Connector_PinHeader_2.54mm:PinHeader_1x04_P2.54mm_Vertical
- removed SPI1: SPI, Connector_PinHeader_2.54mm:PinHeader_1x06_P2.54mm_Vertical
- removed SW3: SW_Push, Button_Switch_THT:SW_PUSH_6mm
- removed the U3 at (165.1, 38.1)
- added BUTTON: ~, Connector_PinHeader_2.54mm:PinHeader_1x02_P2.54mm_Vertical, F.Cu at (137.9, 141.0)
- added DS1: WC1602A, Display:WC1602A, F.Cu at (70.9, 27.8)
- added I2C: I2C, Connector_PinHeader_2.54mm:PinHeader_1x04_P2.54mm_Vertical, F.Cu at (141.0, 83.9)
- added JP4: SolderJumper_2_Open, Jumper:SolderJumper-2_P1.3mm_Open_RoundedPad1.0x1.5mm, F.Cu at (113.9, 104.0)
- added RESET: SW_Push, Button_Switch_THT:SW_PUSH_6mm, F.Cu at (62.8, 146.6)
- added RS485: SolderJumper_2_Open, Jumper:SolderJumper-2_P1.3mm_Open_RoundedPad1.0x1.5mm, F.Cu at (110.4, 104.0)
- added SERIAL: Serial, Connector_PinHeader_2.54mm:PinHeader_1x04_P2.54mm_Vertical, F.Cu at (62.4, 130.7)
- added SPI: SPI, Connector_PinHeader_2.54mm:PinHeader_1x06_P2.54mm_Vertical, F.Cu at (128.2, 133.5)
- added U2: PCF8574AP, AA:PCF8574, F.Cu at (105.0, 81.8)
- H1, H2, H3, H4: footprint MountingHole:MountingHole_2.5mm -> MountingHole:MountingHole_3.5mm
- moved H3 261.0 mm to (48.0, 167.0)
- moved H1 226.3 mm to (48.0, 24.0)
- moved R11 174.4 mm to (67.3, 146.1), turned to -90 degrees
- moved H4 167.0 mm to (162.0, 167.0)
- moved H2 112.4 mm to (162.0, 24.0)
- moved EKSTERNAL 88.5 mm to (141.0, 94.0), turned to 180 degrees
- moved R8 76.2 mm to (128.3, 139.7)
- moved R10 66.6 mm to (149.3, 145.1), turned to -90 degrees
- moved U1 66.5 mm to (125.7, 125.2)
- moved LED2 66.3 mm to (126.7, 95.9), turned to 90 degrees
- moved LM1 64.5 mm to (93.5, 138.2)
- moved R4 62.3 mm to (68.3, 130.5), turned to -90 degrees
- moved U3 61.4 mm to (68.6, 83.8), turned to -90 degrees
- moved LED1 60.7 mm to (122.2, 95.9), turned to 90 degrees
- moved D2 60.6 mm to (113.0, 96.5), turned to 180 degrees
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- renumbered EKSTERNAL1 to EKSTERNAL, JP1 to LED1, JP2 to LED2, LM2596 to LM1, MAX485 to MAX1, R14 to R1, R11 to R10, R10 to R11, R13 to R2, R2 to R3, R6 to R4, R1 to R5, R12 to R6, R3 to R7, R5 to R8, R4 to R9, RN2 to RN1, RS485 to RS, U4 to U1, U2 to U3
Connections:
- LM1 pad 1: Net-(LM2596-IN+) -> unconnected-(LM1-IN+-Pad1)
- LM1 pad 2: Net-(LM2596-IN-) -> unconnected-(LM1-IN--Pad2)
- MAX1 pad 2: Net-(MAX485-A) -> Net-(MAX1-A)
- MAX1 pad 3: Net-(MAX485-B) -> Net-(MAX1-B)
- MAX1 pad 8: Net-(MAX485-DI) -> Net-(JP4-B)
- R3 pad 2: Net-(SERIAL1-Pin_3) -> Net-(JP1-B)
- R4 pad 1: Net-(SERIAL1-Pin_3) -> Net-(JP1-B)
- RN1 pad 1: unconnected-(RN2-common-Pad1) -> +5V
- RN1 pad 10: unconnected-(RN2-R9-Pad10) -> Net-(DS1-D7)
- RN1 pad 3: unconnected-(RN2-R2-Pad3) -> Net-(DS1-RS)
- RN1 pad 4: unconnected-(RN2-R3-Pad4) -> Net-(DS1-R/W)
- RN1 pad 5: unconnected-(RN2-R4-Pad5) -> Net-(DS1-E)
- RN1 pad 7: unconnected-(RN2-R6-Pad7) -> Net-(DS1-D4)
- RN1 pad 8: unconnected-(RN2-R7-Pad8) -> Net-(DS1-D5)
- RN1 pad 9: unconnected-(RN2-R8-Pad9) -> Net-(DS1-D6)
- RS pad 2: Net-(MAX485-B) -> Net-(MAX1-A)
- RS pad 3: Net-(MAX485-A) -> Net-(MAX1-B)
- U1 pad 15: Net-(SERIAL1-Pin_3) -> Net-(JP1-A)
- U1 pad 16: Net-(MAX485-DI) -> Net-(JP4-A)
- U3 pad 2: +5V -> (no net)
Routing:
- net +5V: track 0.00 -> 292.9 mm
- net +3.3V: track 0.00 -> 226.9 mm
- net /SCL: track 0.00 -> 121.0 mm
- net /SDA: track 0.00 -> 114.9 mm
- net Net-(JP1-A): track 0.00 -> 93.0 mm, vias 0 -> 1
- net Net-(JP4-A): track 0.00 -> 88.9 mm
- net /RST: track 0.00 -> 88.9 mm
- net Net-(DS1-RS): track 0.00 -> 73.9 mm
- net Net-(DS1-E): track 0.00 -> 73.9 mm
- net Net-(DS1-R/W): track 0.00 -> 73.9 mm
- net Net-(DS1-D6): track 0.00 -> 70.9 mm
- net Net-(DS1-D5): track 0.00 -> 70.9 mm
- net Net-(DS1-D4): track 0.00 -> 70.9 mm
- net Net-(DS1-D7): track 0.00 -> 70.9 mm
- net Net-(JP1-B): track 0.00 -> 68.1 mm, vias 0 -> 1
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- added copper zone on B.Cu, net (none)
- added copper zone on F.Cu, net (none)
- added copper zone on B.Cu, net GND
- added copper zone on F.Cu, net GND
Other:
- board outline added: 122 x 151 mm
- board text added: "+5V"
- board text added: "A"
- board text added: "B"
- board text added: "CS"
- board text added: "D3"
- board text added: "D4"
- board text added: "EMBEDDED SYSTEM PLATFORM MODULE Version 1.0 12-10-2026"
- board text added: "GND"
- board text added: "MISO"
- board text added: "MOSI"
- board text added: "RX"
- board text added: "SCK"
- board text added: "SCL"
- board text added: "SDA"
- board text added: "SW1"
- board text added: "SW2"
- board text added: "TX"
