File: Capstone/Capstone.kicad_sch (KiCad schematic)
At the start: 36 parts, among them SW1 SW_Push, SW2 SW_Push, SW3 SW_Push, U2 DS3231M, U3 PCF8574AP, U4 WEMOS_D1_mini

Commit message: First Commit
Parts:
- removed DS1: HY1602E, Display:HY1602E, symbol Display_Character:HY1602E
- removed LM2596_E1: LM2596, Connector_PinHeader_2.54mm:PinHeader_1x04_P2.54mm_Vertical, symbol Connector_Generic:Conn_01x02
- removed U3: PCF8574AP, AA:MODULE_LCD-16X2, symbol Interface_Expansion:PCF8574AP
- added DS1: WC1602A, Display:WC1602A, symbol Display_Character:WC1602A
- added JP1, JP4: SolderJumper_2_Open, Jumper:SolderJumper-2_P1.3mm_Open_RoundedPad1.0x1.5mm, symbol Jumper:SolderJumper_2_Open
- added U2: PCF8574AP, AA:PCF8574, symbol Interface_Expansion:PCF8574AP
- BUTTON1: value Button -> (none); footprint Connector_PinHeader_2.54mm:PinHeader_1x04_P2.54mm_Vertical -> Connector_PinHeader_2.54mm:PinHeader_1x02_P2.54mm_Vertical
- H1, H2, H3, H4: footprint MountingHole:MountingHole_2.5mm -> MountingHole:MountingHole_3.5mm
- renumbered JP1 to JP2, JP2 to JP3, LM2596 to LM1, MAX485 to MAX1, R14 to R1, R11 to R10, R10 to R11, R13 to R2, R2 to R3, R6 to R4, R1 to R5, R12 to R6, R3 to R7, R5 to R8, R4 to R9, RN2 to RN1, RS485 to RS1, U4 to U1, U2 to U3
Connections:
- net +3.3V: now also U2.16 (VDD)
- net +5V: now also RN1.1 (common), DS1.2 (VDD)
- net GND: now also DS1.1 (VSS), U2.8 (GND)
- net SCL: now also U2.14 (SCL)
- net SDA: now also U2.15 (SDA)
- net at SERIAL1.2 (Pin_2), U1.16 (TX): now also JP4.1 (A); no longer MAX1.8 (DI)
- net at RN1.7 (R6): now also DS1.11 (D4), U2.9 (P4)
- net at RN1.8 (R7): now also DS1.12 (D5), U2.10 (P5)
- net at RN1.9 (R8): now also DS1.13 (D6), U2.11 (P6)
- net at RN1.10 (R9): now also DS1.14 (D7), U2.12 (P7)
- net at SERIAL1.3 (Pin_3), U1.15 (RX): now also JP1.1 (A); no longer R3.2, R4.1
- net at RN1.3 (R2): now also DS1.4 (RS), U2.4 (P0)
- net at RN1.4 (R3): now also DS1.5 (R/W), U2.5 (P1)
- net at RN1.5 (R4): now also DS1.6 (E), U2.6 (P2)
- new net: JP1.2 (B), R3.2, R4.1
- new net: JP4.2 (B), MAX1.8 (DI)
- no-connect marks 8 -> 20
Other:
- moved on the sheet: BUTTON1, D1, D2, EKSTERNAL1, H1, H2, H3, H4, I2C1, JP2, JP3, LM1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
